File: Receivers and Transmitters/Receivers/Antenna Diversity/ExpressLRS_2.4GHz/AD1_2.4G/SE2431L.kicad_sch (KiCad schematic)
At the start: 8 parts, among them U4 SE2431L-R

Commit message: Update Antenna Diversity (AD1_2.4G), True Antenna Diversity (TD1_2.4G), and Gemini Mode transmitter (G_TX1): Modify KiCad files, add BOMs and production files; update images, docs, videos, and README; remove outdated Mechanical CAD file
Parts:
- C4, C5, C6, C7: footprint Capacitor_SMD:C_0805_2012Metric_Pad1.18x1.45mm_HandSolder -> Capacitor_SMD:C_0603_1608Metric_Pad1.08x0.95mm_HandSolder
- R1, R10, R9: footprint Resistor_SMD:R_0805_2012Metric_Pad1.20x1.40mm_HandSolder -> Resistor_SMD:R_0603_1608Metric_Pad0.98x0.95mm_HandSolder
Other:
- company: https://github.com/Paschalis | TeodoraMiu -> https://github.com/Paschalis
