File: Receivers and Transmitters/Receivers/Antenna Diversity/ExpressLRS_2.4GHz/AD1_2.4G/SX1280.kicad_sch (KiCad schematic)
At the start: 8 parts, among them U2 SX1280IMLTRT, Y1 52MHz

Commit message: Update Antenna Diversity (AD1_2.4G), True Antenna Diversity (TD1_2.4G), and Gemini Mode transmitter (G_TX1): Modify KiCad files, add BOMs and production files; update images, docs, videos, and README; remove outdated Mechanical CAD file
Parts:
- C16, C17, C18, C19, C20: footprint Capacitor_SMD:C_0805_2012Metric_Pad1.18x1.45mm_HandSolder -> Capacitor_SMD:C_0603_1608Metric_Pad1.08x0.95mm_HandSolder
Other:
- company: https://github.com/Paschalis | TeodoraMiu -> https://github.com/Paschalis
Changed lines of the file:
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@@
 (kicad_sch
-	(version 20231120)
+	(version 20250114)
 	(generator "eeschema")
-	(generator_version "8.0")
+	(generator_version "9.0")
 	(paper "A4")
 	(title_block
 		(date "05-01-2025")
 		(rev "1.0")
-		(company "https://github.com/Paschalis | TeodoraMiu")
+		(company "https://github.com/Paschalis")
 		(comment 2 "capabilities in LoRa communication, making it ideal for reliable telemetry.")
 		(comment 3 "The SX1280 is used for its long-range, low-power, and high-performance ")
+	)
+	(rectangle
+		(start 176.53 41.91)
+		(end 278.13 129.54)
+		(stroke
+			(width 0)
+			(type dash)
+		)
+		(fill
+			(type none)
+		)
+	)
+	(rectangle
+		(start 21.59 43.18)
+		(end 167.64 114.3)
+		(stroke
+			(width 0)
+			(type dash)
+		)
+		(fill
+			(type none)
+		)
+	)
+	(text "2.45GHz Impedance Matched Low Pass Filter Optimized for Semtech SX1280 and SX1281 chipsets"
+		(exclude_from_sim no)
+		(at 227.838 122.682 0)
+		(effects
+			(font
+				(size 1.27 1.27)
+			)
+		)
+	)
+	(text "2450FM07D0034001T (LOW PASS FILTER)"
+		(exclude_from_sim no)
+		(at 207.772 40.132 0)
+		(effects
+			(font
+				(size 2 2)
+			)
+		)
+	)
+	(text "Paschalis M."
+		(exclude_from_sim no)
+		(at 214.376 183.388 0)
+		(effects
+			(font
+				(size 1.27 1.27)
+			)
+		)
+	)
+	(text "LoRa Connect RF Transceiver SX1280"
+		(exclude_from_sim no)
+		(at 50.038 41.148 0)
+		(effects
+			(font
+				(size 2 2)
+			)
+		)
 	)
 	(junction
@@
 		)
 	)
-	(rectangle
-		(start 176.53 41.91)
-		(end 278.13 129.54)
-		(stroke
-			(width 0)
-			(type dash)
-		)
-		(fill
-			(type none)
-		)
-	)
-	(rectangle
-		(start 21.59 43.18)
-		(end 167.64 114.3)
-		(stroke
-			(width 0)
-			(type dash)
-		)
-		(fill
-			(type none)
-		)
-	)
-	(text "2.45GHz Impedance Matched Low Pass Filter Optimized for Semtech SX1280 and SX1281 chipsets"
-		(exclude_from_sim no)
-		(at 227.838 122.682 0)
+	(label "RFIO"
+		(at 210.82 82.55 180)
+		(effects
+			(font
+				(size 1 1)
+			)
+			(justify right bottom)
+		)
+	)
+	(label "VDD_INN"
+		(at 68.58 66.04 180)
+		(effects
+			(font
+				(size 1 1)
+			)
+			(justify right bottom)
+		)
+	)
+	(label "RFIO"
+		(at 130.81 71.12 0)
+		(effects
+			(font
+				(size 1 1)
+			)
+			(justify left bottom)
+		)
+	)
+	(label "VDD_INN"
+		(at 59.69 91.44 180)
+		(effects
+			(font
+				(size 1 1)
+			)
+			(justify right bottom)
+		)
+	)
+	(hierarchical_label "SX_SCK"
+		(shape input)
+		(at 130.81 81.28 0)
 		(effects
 			(font
 				(size 1.27 1.27)
 			)
-		)
-	)
-	(text "2450FM07D0034001T (LOW PASS FILTER)"
-		(exclude_from_sim no)
-		(at 207.772 40.132 0)
-		(effects
-			(font
-				(size 2 2)
-			)
-		)
-	)
-	(text "Paschalis M."
-		(exclude_from_sim no)
-		(at 214.376 183.388 0)
+			(justify left)
+		)
+	)
+	(hierarchical_label "NSS_CTS"
+		(shape input)
+		(at 130.81 78.74 0)
 		(effects
 			(font
 				(size 1.27 1.27)
 			)
-		)
-	)
-	(text "LoRa Connect RF Transceiver SX1280"
-		(exclude_from_sim no)
-		(at 50.038 41.148 0)
-		(effects
-			(font
-				(size 2 2)
-			)
-		)
-	)
-	(label "RFIO"
-		(at 210.82 82.55 180)
-		(fields_autoplaced yes)
-		(effects
-			(font
-				(size 1 1)
-			)
-			(justify right bottom)
-		)
-	)
-	(label "VDD_INN"
-		(at 68.58 66.04 180)
-		(fields_autoplaced yes)
-		(effects
-			(font
-				(size 1 1)
-			)
-			(justify right bottom)
-		)
-	)
-	(label "RFIO"
-		(at 130.81 71.12 0)
-		(fields_autoplaced yes)
-		(effects
-			(font
-				(size 1 1)
-			)
-			(justify left bottom)
-		)
-	)
-	(label "VDD_INN"
-		(at 59.69 91.44 180)
-		(fields_autoplaced yes)
-		(effects
-			(font
-				(size 1 1)
-			)
-			(justify right bottom)
-		)
-	)
-	(hierarchical_label "SX_SCK"
+			(justify left)
+		)
+	)
+	(hierarchical_label "SX_NRESET"
 		(shape input)
-		(at 130.81 81.28 0)
-		(fields_autoplaced yes)
+		(at 68.58 68.58 180)
 		(effects
 			(font
 				(size 1.27 1.27)
 			)
-			(justify left)
-		)
-	)
-	(hierarchical_label "NSS_CTS"
-		(shape input)
-		(at 130.81 78.74 0)
-		(fields_autoplaced yes)
+			(justify right)
+		)
+	)
+	(hierarchical_label "BUSY"
+		(shape output)
+		(at 68.58 78.74 180)
 		(effects
 			(font
 				(size 1.27 1.27)
 			)
-			(justify left)
-		)
-	)
-	(hierarchical_label "SX_NRESET"
-		(shape input)
-		(at 68.58 68.58 180)
-		(fields_autoplaced yes)
+			(justify right)
+		)
+	)
+	(hierarchical_label "TR"
+		(shape output)
+		(at 246.38 82.55 0)
 		(effects
 			(font
 				(size 1.27 1.27)
 			)
-			(justify right)
-		)
-	)
-	(hierarchical_label "BUSY"
+			(justify left)
+		)
+	)
+	(hierarchical_label "SX_MISO"
 		(shape output)
-		(at 68.58 78.74 180)
-		(fields_autoplaced yes)
+		(at 130.81 86.36 0)
 		(effects
 			(font
 				(size 1.27 1.27)
 			)
-			(justify right)
-		)
-	)
-	(hierarchical_label "TR"
-		(shape output)
-		(at 246.38 82.55 0)
-		(fields_autoplaced yes)
+			(justify left)
+		)
+	)
+	(hierarchical_label "SX_MOSI"
+		(shape input)
+		(at 130.81 83.82 0)
 		(effects
 			(font
@@
 		)
 	)
-	(hierarchical_label "SX_MISO"
-		(shape output)
-		(at 130.81 86.36 0)
-		(fields_autoplaced yes)
-		(effects
-			(font
-				(size 1.27 1.27)
-			)
-			(justify left)
-		)
-	)
-	(hierarchical_label "SX_MOSI"
-		(shape input)
-		(at 130.81 83.82 0)
-		(fields_autoplaced yes)
-		(effects
-			(font
-				(size 1.27 1.27)
-			)
-			(justify left)
-		)
-	)
 	(hierarchical_label "DIO1"
 		(shape bidirectional)
 		(at 68.58 81.28 180)
-		(fields_autoplaced yes)
 		(effects
 			(font
@@
 			)
 		)
-		(property "Footprint" "Capacitor_SMD:C_0805_2012Metric_Pad1.18x1.45mm_HandSolder"
+		(property "Footprint" "Capacitor_SMD:C_0603_1608Metric_Pad1.08x0.95mm_HandSolder"
 			(at 48.26 96.52 0)
 			(effects
@@
 			)
 		)
-		(property "Footprint" "Capacitor_SMD:C_0805_2012Metric_Pad1.18x1.45mm_HandSolder"
+		(property "Footprint" "Capacitor_SMD:C_0603_1608Metric_Pad1.08x0.95mm_HandSolder"
 			(at 62.23 96.52 0)
 			(effects
@@
 			)
 		)
-		(property "Footprint" "Capacitor_SMD:C_0805_2012Metric_Pad1.18x1.45mm_HandSolder"
+		(property "Footprint" "Capacitor_SMD:C_0603_1608Metric_Pad1.08x0.95mm_HandSolder"
 			(at 57.15 63.5 0)
 			(effects
@@
 			)
 		)
-		(property "Footprint" "Capacitor_SMD:C_0805_2012Metric_Pad1.18x1.45mm_HandSolder"
+		(property "Footprint" "Capacitor_SMD:C_0603_1608Metric_Pad1.08x0.95mm_HandSolder"
 			(at 71.12 96.52 0)
 			(effects
@@
 			)
 		)
-		(property "Footprint" "Capacitor_SMD:C_0805_2012Metric_Pad1.18x1.45mm_HandSolder"
+		(property "Footprint" "Capacitor_SMD:C_0603_1608Metric_Pad1.08x0.95mm_HandSolder"
 			(at 146.05 92.71 0)
 			(effects
