File: Receivers and Transmitters/Receivers/True Antenna Diversity/ExpressLRS_2.4GHz/TD1_2.4G/RFX2401C_ANT2.kicad_sch (KiCad schematic)
At the start: 7 parts, among them U6 RFX2401C, U7 2450LP14B100

Commit message: Updated schematics for TD1_2.4G receiver: ESP32, SX1280, and RFX2401C blocks
Other:
- company: https://github.com/Paschalis | TeodoraMiu -> https://github.com/Paschalis
Changed lines of the file:
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@@
 		(date "2025-02-23")
 		(rev "1.0")
-		(company "https://github.com/Paschalis | TeodoraMiu")
+		(company "https://github.com/Paschalis")
 	)
 	(rectangle
